File: hardware/controls.sch (KiCad schematic (older format))
At the start: 7 parts

Commit message: four inputs mapped out with footprints
Parts:
- added C? (x3): 330pF, symbol C
- added J? (x3): PJ301M-12, symbol PJ301M-12
- added R? (x3): 1k, Resistors_SMD:R_0805_HandSoldering, symbol R
- added R? (x3): 499, Resistors_SMD:R_0805_HandSoldering, symbol R
- added R? (x3): 270, Resistors_SMD:R_0805_HandSoldering, symbol R
- added R? (x3): 100R, Resistors_SMD:R_0805_HandSoldering, symbol R
- added unit 2 of U301
- added unit 4 of U301
- added unit 3 of U301
- U301: renamed from U?; footprint (none) -> Housings_DIP:DIP-14_W7.62mm
- gave numbers to parts that had none: 6
Connections:
- net +5V: now also U301.4 (V+), U301.4 (V+), U301.4 (V+)
- net -5V: now also R?.2, R?.2, R?.2
- net Earth: now also J?.1, J?.1, J?.1, J?.2, J?.2, J?.2, U301.10 (+), U301.11 (V-), U301.11 (V-), U301.11 (V-), U301.12 (+), U301.5 (+)
- new net: J?.3, R?.2 (x3)
- new net: C?.2, R?.1, R?.1, R?.2, U301.6 (-)
- new net: C?.1, R?.1, R?.2, U301.7
- new net: C?.2, R?.1, R?.1, R?.2, U301.9 (-)
- new net: C?.1, R?.1, R?.2, U301.8
- new net: C?.2, R?.1, R?.1, R?.2, U301.13 (-)
- new net: C?.1, R?.1, R?.2, U301.14
- new net CV2: R?.1
- new net CV3: R?.1
- new net CV4: R?.1
