File: hardware/jacks 1-4.sch (KiCad schematic (older format))
At the start: 25 parts, among them J301 PJ301M-12, J302 PJ301M-12, J303 PJ301M-12, J304 PJ301M-12, U301 MCP6004

Commit message: jacks on a different sheet than the buffers. single PCB with jumpers and mouse bites
Parts:
- added P?: CONN_01X06, Pin_Headers:Pin_Header_Straight_1x06_Pitch2.54mm, symbol CONN_01X06
- C301, C302, C303, C304: value 330pF -> 560pF; footprint (none) -> Capacitors_THT:C_Axial_L3.8mm_D2.6mm_P7.50mm_Horizontal
Connections:
- wire segments 80 -> 112
Changed lines of the file:
@@
 $Descr A4 11693 8268
 encoding utf-8
-Sheet 3 4
+Sheet 3 5
 Title ""
 Date ""
@@
 	2000 1800 2250 1800
 Wire Wire Line
-	2250 1800 2250 2350
+	2250 1800 2250 1950
+Wire Wire Line
+	2250 1950 2250 2350
 Wire Wire Line
 	2000 1950 2250 1950
@@
 	2650 1350 2900 1350
 Wire Wire Line
-	2900 1350 2900 2700
-Wire Wire Line
-	2650 1700 3150 1700
+	2900 1350 2900 1700
+Wire Wire Line
+	2900 1700 2900 2300
+Wire Wire Line
+	2900 2300 2900 2700
+Wire Wire Line
+	2650 1700 2900 1700
+Wire Wire Line
+	2900 1700 3150 1700
 Connection ~ 2900 1700
 $Comp
@@
 P 3400 2300
 F 0 "C301" V 3450 2350 50  0000 L CNN
-F 1 "330pF" V 3350 2350 50  0000 L CNN
-F 2 "" H 3438 2150 50  0000 C CNN
+F 1 "560pF" V 3350 2350 50  0000 L CNN
+F 2 "Capacitors_THT:C_Axial_L3.8mm_D2.6mm_P7.50mm_Horizontal" H 3438 2150 50  0001 C CNN
 F 3 "" H 3400 2300 50  0000 C CNN
 	1    3400 2300
@@
 $EndComp
 Wire Wire Line
-	3750 1600 4150 1600
+	3750 1600 3950 1600
+Wire Wire Line
+	3950 1600 4150 1600
 Wire Wire Line
 	3550 2300 3950 2300
 Wire Wire Line
-	3950 1600 3950 2700
+	3950 1600 3950 2300
+Wire Wire Line
+	3950 2300 3950 2700
 Connection ~ 3950 1600
 Wire Wire Line
@@
 	6950 1800 7200 1800
 Wire Wire Line
-	7200 1800 7200 2350
+	7200 1800 7200 1950
+Wire Wire Line
+	7200 1950 7200 2350
 Wire Wire Line
 	6950 1950 7200 1950
@@
 	7600 1350 7850 1350
 Wire Wire Line
-	7850 1350 7850 2700
-Wire Wire Line
-	7600 1700 8100 1700
+	7850 1350 7850 1700
+Wire Wire Line
+	7850 1700 7850 2300
+Wire Wire Line
+	7850 2300 7850 2700
+Wire Wire Line
+	7600 1700 7850 1700
+Wire Wire Line
+	7850 1700 8100 1700
 Connection ~ 7850 1700
 $Comp
@@
 P 8350 2300
 F 0 "C302" V 8400 2350 50  0000 L CNN
-F 1 "330pF" V 8300 2350 50  0000 L CNN
-F 2 "" H 8388 2150 50  0000 C CNN
+F 1 "560pF" V 8300 2350 50  0000 L CNN
+F 2 "Capacitors_THT:C_Axial_L3.8mm_D2.6mm_P7.50mm_Horizontal" H 8388 2150 50  0001 C CNN
 F 3 "" H 8350 2300 50  0000 C CNN
 	1    8350 2300
@@
 $EndComp
 Wire Wire Line
-	8700 1600 9100 1600
+	8700 1600 8900 1600
+Wire Wire Line
+	8900 1600 9100 1600
 Wire Wire Line
 	8500 2300 8900 2300
 Wire Wire Line
-	8900 1600 8900 2700
+	8900 1600 8900 2300
+Wire Wire Line
+	8900 2300 8900 2700
 Connection ~ 8900 1600
 Wire Wire Line
@@
 	2000 4050 2250 4050
 Wire Wire Line
-	2250 4050 2250 4600
+	2250 4050 2250 4200
+Wire Wire Line
+	2250 4200 2250 4600
 Wire Wire Line
 	2000 4200 2250 4200
@@
 	2650 3600 2900 3600
 Wire Wire Line
-	2900 3600 2900 4950
-Wire Wire Line
-	2650 3950 3150 3950
+	2900 3600 2900 3950
+Wire Wire Line
+	2900 3950 2900 4550
+Wire Wire Line
+	2900 4550 2900 4950
+Wire Wire Line
+	2650 3950 2900 3950
+Wire Wire Line
+	2900 3950 3150 3950
 Connection ~ 2900 3950
 $Comp
@@
 P 3400 4550
 F 0 "C303" V 3450 4600 50  0000 L CNN
-F 1 "330pF" V 3350 4600 50  0000 L CNN
-F 2 "" H 3438 4400 50  0000 C CNN
+F 1 "560pF" V 3350 4600 50  0000 L CNN
+F 2 "Capacitors_THT:C_Axial_L3.8mm_D2.6mm_P7.50mm_Horizontal" H 3438 4400 50  0001 C CNN
 F 3 "" H 3400 4550 50  0000 C CNN
 	1    3400 4550
@@
 $EndComp
 Wire Wire Line
-	3750 3850 4150 3850
+	3750 3850 3950 3850
+Wire Wire Line
+	3950 3850 4150 3850
 Wire Wire Line
 	3550 4550 3950 4550
 Wire Wire Line
-	3950 3850 3950 4950
+	3950 3850 3950 4550
+Wire Wire Line
+	3950 4550 3950 4950
 Connection ~ 3950 3850
 Wire Wire Line
@@
 	6950 4050 7200 4050
 Wire Wire Line
-	7200 4050 7200 4600
+	7200 4050 7200 4200
+Wire Wire Line
+	7200 4200 7200 4600
 Wire Wire Line
 	6950 4200 7200 4200
@@
 	7600 3600 7850 3600
 Wire Wire Line
-	7850 3600 7850 4950
-Wire Wire Line
-	7600 3950 8100 3950
+	7850 3600 7850 3950
+Wire Wire Line
+	7850 3950 7850 4550
+Wire Wire Line
+	7850 4550 7850 4950
+Wire Wire Line
+	7600 3950 7850 3950
+Wire Wire Line
+	7850 3950 8100 3950
 Connection ~ 7850 3950
 $Comp
@@
 P 8350 4550
 F 0 "C304" V 8400 4600 50  0000 L CNN
-F 1 "330pF" V 8300 4600 50  0000 L CNN
-F 2 "" H 8388 4400 50  0000 C CNN
+F 1 "560pF" V 8300 4600 50  0000 L CNN
+F 2 "Capacitors_THT:C_Axial_L3.8mm_D2.6mm_P7.50mm_Horizontal" H 8388 4400 50  0001 C CNN
 F 3 "" H 8350 4550 50  0000 C CNN
 	1    8350 4550
@@
 $EndComp
 Wire Wire Line
-	8700 3850 9100 3850
+	8700 3850 8900 3850
+Wire Wire Line
+	8900 3850 9100 3850
 Wire Wire Line
 	8500 4550 8900 4550
 Wire Wire Line
-	8900 3850 8900 4950
+	8900 3850 8900 4550
+Wire Wire Line
+	8900 4550 8900 4950
 Connection ~ 8900 3850
 Wire Wire Line
@@
 	1    0    0    -1
 $EndComp
+$Comp
+L CONN_01X06 P?
+U 1 1 5BE4B196
+P 1900 6550
+F 0 "P?" H 1900 6900 50  0000 C CNN
+F 1 "CONN_01X06" V 2000 6550 50  0000 C CNN
+F 2 "Pin_Headers:Pin_Header_Straight_1x06_Pitch2.54mm" V 2100 6550 50  0000 C CNN
+F 3 "" H 1900 6550 50  0000 C CNN
+	1    1900 6550
+	1    0    0    -1
+$EndComp
+$Comp
+L +5V #PWR?
+U 1 1 5BE4B7BC
+P 1600 6200
+F 0 "#PWR?" H 1600 6050 50  0001 C CNN
+F 1 "+5V" H 1600 6340 50  0000 C CNN
+F 2 "" H 1600 6200 50  0000 C CNN
+F 3 "" H 1600 6200 50  0000 C CNN
+	1    1600 6200
+	1    0    0    -1
+$EndComp
+Text HLabel 1600 6400 0    60   Input ~ 0
+CV1
+Wire Wire Line
+	1600 6200 1600 6300
+Wire Wire Line
+	1600 6300 1700 6300
+Wire Wire Line
+	1600 6400 1700 6400
+Text HLabel 1600 6500 0    60   Input ~ 0
+CV2
+Text HLabel 1600 6600 0    60   Input ~ 0
+CV3
+Text HLabel 1600 6700 0    60   Input ~ 0
+CV4
+$Comp
+L Earth #PWR?
+U 1 1 5BE4BF98
+P 1600 6900
+F 0 "#PWR?" H 1600 6650 50  0001 C CNN
+F 1 "Earth" H 1600 6750 50  0001 C CNN
+F 2 "" H 1600 6900 50  0000 C CNN
+F 3 "" H 1600 6900 50  0000 C CNN
+	1    1600 6900
+	1    0    0    -1
+$EndComp
+Wire Wire Line
+	1700 6800 1600 6800
+Wire Wire Line
+	1600 6800 1600 6900
+Wire Wire Line
+	1600 6700 1700 6700
+Wire Wire Line
+	1700 6600 1600 6600
+Wire Wire Line
+	1600 6500 1700 6500
 $EndSCHEMATC
