File: hardware/CV jacks.sch (KiCad schematic (older format))
At the start: 8 parts, among them J501 PJ301M-12, J502 PJ301M-12, J503 PJ301M-12, J504 PJ301M-12, J505 PJ301M-12, J506 PJ301M-12, J507 PJ301M-12, J508 PJ301M-12

Commit message: reworked input board
Parts:
- added EXPANDER501: CONN_02X05, Pin_Headers:Pin_Header_Straight_2x05_Pitch2.54mm, symbol CONN_02X05
Connections:
- net Earth: now also EXPANDER501.9 (P9); no longer J501.2, J502.2, J503.2, J504.2, J505.2, J506.2, J507.2, J508.2
- new net expansion1: EXPANDER501.1 (P1), J501.2
- new net expansion2: EXPANDER501.3 (P3), J502.2
- new net expansion3: EXPANDER501.5 (P5), J503.2
- new net expansion4: EXPANDER501.7 (P7), J504.2
- new net expansion5: EXPANDER501.8 (P8), J505.2
- new net expansion6: EXPANDER501.6 (P6), J506.2
- new net expansion7: EXPANDER501.4 (P4), J507.2
- new net expansion8: EXPANDER501.2 (P2), J508.2
- no-connect marks 0 -> 1
Changed lines of the file:
@@
 $EndComp
-Wire Wire Line
-	2100 1200 2100 1350
 Wire Wire Line
 	2100 1350 2200 1350
@@
 $EndComp
 Wire Wire Line
-	2100 1900 2100 2050
-Wire Wire Line
 	2100 2050 2200 2050
 $Comp
@@
 $EndComp
 Wire Wire Line
-	2100 2600 2100 2750
-Wire Wire Line
 	2100 2750 2200 2750
 $Comp
@@
 $EndComp
 Wire Wire Line
-	2100 3300 2100 3450
-Wire Wire Line
 	2100 3450 2200 3450
 $Comp
@@
 $EndComp
 Wire Wire Line
-	2100 4000 2100 4150
-Wire Wire Line
 	2100 4150 2200 4150
 $Comp
@@
 $EndComp
 Wire Wire Line
-	2100 4700 2100 4850
-Wire Wire Line
 	2100 4850 2200 4850
 $Comp
@@
 $EndComp
 Wire Wire Line
-	2100 5400 2100 5550
-Wire Wire Line
 	2100 5550 2200 5550
 $Comp
@@
 $EndComp
 Wire Wire Line
-	2100 6100 2100 6250
-Wire Wire Line
 	2100 6250 2200 6250
+$Comp
+L CONN_02X05 EXPANDER501
+U 1 1 5C0083CE
+P 4700 3550
+F 0 "EXPANDER501" H 4700 3850 50  0000 C CNN
+F 1 "CONN_02X05" H 4700 3250 50  0000 C CNN
+F 2 "Pin_Headers:Pin_Header_Straight_2x05_Pitch2.54mm" H 4700 2350 50  0001 C CNN
+F 3 "" H 4700 2350 50  0000 C CNN
+	1    4700 3550
+	1    0    0    -1
+$EndComp
+Text Label 4450 3350 2    60   ~ 0
+expansion1
+Text Label 4450 3450 2    60   ~ 0
+expansion2
+Text Label 4450 3550 2    60   ~ 0
+expansion3
+Text Label 4450 3650 2    60   ~ 0
+expansion4
+Text Label 4950 3650 0    60   ~ 0
+expansion5
+Text Label 4950 3550 0    60   ~ 0
+expansion6
+Text Label 4950 3450 0    60   ~ 0
+expansion7
+Text Label 4950 3350 0    60   ~ 0
+expansion8
+Text Label 2800 1200 0    60   ~ 0
+expansion1
+Wire Wire Line
+	2100 1200 2800 1200
+Wire Wire Line
+	2100 1900 2800 1900
+Text Label 2800 1900 0    60   ~ 0
+expansion2
+Text Label 2800 2600 0    60   ~ 0
+expansion3
+Text Label 2800 3300 0    60   ~ 0
+expansion4
+Text Label 2800 4000 0    60   ~ 0
+expansion5
+Text Label 2800 4700 0    60   ~ 0
+expansion6
+Text Label 2800 5400 0    60   ~ 0
+expansion7
+Text Label 2800 6100 0    60   ~ 0
+expansion8
+Wire Wire Line
+	2100 2600 2800 2600
+Wire Wire Line
+	2100 3300 2800 3300
+Wire Wire Line
+	2100 4000 2800 4000
+Wire Wire Line
+	2100 4700 2800 4700
+Wire Wire Line
+	2100 5400 2800 5400
+Wire Wire Line
+	2100 6100 2800 6100
+$Comp
+L Earth #PWR062
+U 1 1 5C008C4D
+P 3950 3750
+F 0 "#PWR062" H 3950 3500 50  0001 C CNN
+F 1 "Earth" H 3950 3600 50  0001 C CNN
+F 2 "" H 3950 3750 50  0000 C CNN
+F 3 "" H 3950 3750 50  0000 C CNN
+	1    3950 3750
+	0    1    1    0
+$EndComp
+NoConn ~ 4950 3750
+Wire Wire Line
+	4450 3750 3950 3750
 $EndSCHEMATC
