File: hardware/buffers 5-6.sch (KiCad schematic (older format))
At the start: 21 parts, among them U601 MCP6004

Commit message: most of the scematic is complete with the exception of the -5V offset
Parts:
- U601: footprint Housings_DIP:DIP-14_W7.62mm -> Housings_SOIC:SOIC-14_3.9x8.7mm_Pitch1.27mm
Changed lines of the file:
@@
 F 0 "U601" H 3400 2450 50  0000 L CNN
 F 1 "MCP6004" H 3400 2050 50  0000 L CNN
-F 2 "Housings_DIP:DIP-14_W7.62mm" H 3350 2350 50  0001 C CNN
+F 2 "Housings_SOIC:SOIC-14_3.9x8.7mm_Pitch1.27mm" H 3350 2350 50  0001 C CNN
 F 3 "" H 3450 2450 50  0000 C CNN
 	1    3400 2250
@@
 	1950 2350 2300 2350
 $Comp
-L +5V #PWR053
+L +5V #PWR064
 U 1 1 5BE53446
 P 3300 1950
-F 0 "#PWR053" H 3300 1800 50  0001 C CNN
+F 0 "#PWR064" H 3300 1800 50  0001 C CNN
 F 1 "+5V" H 3300 2090 50  0000 C CNN
 F 2 "" H 3300 1950 50  0000 C CNN
@@
 $EndComp
 $Comp
-L Earth #PWR054
+L Earth #PWR065
 U 1 1 5BE5344C
 P 3300 2550
-F 0 "#PWR054" H 3300 2300 50  0001 C CNN
+F 0 "#PWR065" H 3300 2300 50  0001 C CNN
 F 1 "Earth" H 3300 2400 50  0001 C CNN
 F 2 "" H 3300 2550 50  0000 C CNN
@@
 Connection ~ 2850 2350
 $Comp
-L Earth #PWR055
+L Earth #PWR066
 U 1 1 5BE53459
 P 3000 1800
-F 0 "#PWR055" H 3000 1550 50  0001 C CNN
+F 0 "#PWR066" H 3000 1550 50  0001 C CNN
 F 1 "Earth" H 3000 1650 50  0001 C CNN
 F 2 "" H 3000 1800 50  0000 C CNN
@@
 	6900 2350 7250 2350
 $Comp
-L +5V #PWR056
+L +5V #PWR067
 U 1 1 5BE5349B
 P 8250 1950
-F 0 "#PWR056" H 8250 1800 50  0001 C CNN
+F 0 "#PWR067" H 8250 1800 50  0001 C CNN
 F 1 "+5V" H 8250 2090 50  0000 C CNN
 F 2 "" H 8250 1950 50  0000 C CNN
@@
 $EndComp
 $Comp
-L Earth #PWR057
+L Earth #PWR068
 U 1 1 5BE534A1
 P 8250 2550
-F 0 "#PWR057" H 8250 2300 50  0001 C CNN
+F 0 "#PWR068" H 8250 2300 50  0001 C CNN
 F 1 "Earth" H 8250 2400 50  0001 C CNN
 F 2 "" H 8250 2550 50  0000 C CNN
@@
 Connection ~ 7800 2350
 $Comp
-L Earth #PWR058
+L Earth #PWR069
 U 1 1 5BE534AE
 P 7950 1800
-F 0 "#PWR058" H 7950 1550 50  0001 C CNN
+F 0 "#PWR069" H 7950 1550 50  0001 C CNN
 F 1 "Earth" H 7950 1650 50  0001 C CNN
 F 2 "" H 7950 1800 50  0000 C CNN
@@
 F 0 "U601" H 8350 2450 50  0000 L CNN
 F 1 "MCP6004" H 8350 2050 50  0000 L CNN
-F 2 "Housings_DIP:DIP-14_W7.62mm" H 8300 2350 50  0001 C CNN
+F 2 "Housings_SOIC:SOIC-14_3.9x8.7mm_Pitch1.27mm" H 8300 2350 50  0001 C CNN
 F 3 "" H 8400 2450 50  0000 C CNN
 	2    8350 2250
@@
 	1950 4600 2300 4600
 $Comp
-L +5V #PWR059
+L +5V #PWR070
 U 1 1 5BE534F7
 P 3300 4200
-F 0 "#PWR059" H 3300 4050 50  0001 C CNN
+F 0 "#PWR070" H 3300 4050 50  0001 C CNN
 F 1 "+5V" H 3300 4340 50  0000 C CNN
 F 2 "" H 3300 4200 50  0000 C CNN
@@
 $EndComp
 $Comp
-L Earth #PWR060
+L Earth #PWR071
 U 1 1 5BE534FD
 P 3300 4800
-F 0 "#PWR060" H 3300 4550 50  0001 C CNN
+F 0 "#PWR071" H 3300 4550 50  0001 C CNN
 F 1 "Earth" H 3300 4650 50  0001 C CNN
 F 2 "" H 3300 4800 50  0000 C CNN
@@
 Connection ~ 2850 4600
 $Comp
-L Earth #PWR061
+L Earth #PWR072
 U 1 1 5BE5350A
 P 3000 4050
-F 0 "#PWR061" H 3000 3800 50  0001 C CNN
+F 0 "#PWR072" H 3000 3800 50  0001 C CNN
 F 1 "Earth" H 3000 3900 50  0001 C CNN
 F 2 "" H 3000 4050 50  0000 C CNN
@@
 	6900 4600 7250 4600
 $Comp
-L +5V #PWR062
+L +5V #PWR073
 U 1 1 5BE5354C
 P 8250 4200
-F 0 "#PWR062" H 8250 4050 50  0001 C CNN
+F 0 "#PWR073" H 8250 4050 50  0001 C CNN
 F 1 "+5V" H 8250 4340 50  0000 C CNN
 F 2 "" H 8250 4200 50  0000 C CNN
@@
 $EndComp
 $Comp
-L Earth #PWR063
+L Earth #PWR074
 U 1 1 5BE53552
 P 8250 4800
-F 0 "#PWR063" H 8250 4550 50  0001 C CNN
+F 0 "#PWR074" H 8250 4550 50  0001 C CNN
 F 1 "Earth" H 8250 4650 50  0001 C CNN
 F 2 "" H 8250 4800 50  0000 C CNN
@@
 Connection ~ 7800 4600
 $Comp
-L Earth #PWR064
+L Earth #PWR075
 U 1 1 5BE5355F
 P 7950 4050
-F 0 "#PWR064" H 7950 3800 50  0001 C CNN
+F 0 "#PWR075" H 7950 3800 50  0001 C CNN
 F 1 "Earth" H 7950 3900 50  0001 C CNN
 F 2 "" H 7950 4050 50  0000 C CNN
@@
 F 0 "U601" H 8350 4700 50  0000 L CNN
 F 1 "MCP6004" H 8350 4300 50  0000 L CNN
-F 2 "Housings_DIP:DIP-14_W7.62mm" H 8300 4600 50  0001 C CNN
+F 2 "Housings_SOIC:SOIC-14_3.9x8.7mm_Pitch1.27mm" H 8300 4600 50  0001 C CNN
 F 3 "" H 8400 4700 50  0000 C CNN
 	4    8350 4500
@@
 F 0 "U601" H 3400 4700 50  0000 L CNN
 F 1 "MCP6004" H 3400 4300 50  0000 L CNN
-F 2 "Housings_DIP:DIP-14_W7.62mm" H 3350 4600 50  0001 C CNN
+F 2 "Housings_SOIC:SOIC-14_3.9x8.7mm_Pitch1.27mm" H 3350 4600 50  0001 C CNN
 F 3 "" H 3450 4700 50  0000 C CNN
 	3    3400 4500

Commit message: updated footprint & first tracks laid
Parts:
- C601, C602, C603, C604: footprint Capacitors_THT:C_Axial_L3.8mm_D2.6mm_P7.50mm_Horizontal -> Capacitors_SMD:C_0805_HandSoldering
Changed lines of the file:
@@
 	1950 2350 2300 2350
 $Comp
-L +5V #PWR064
+L +5V #PWR066
 U 1 1 5BE53446
 P 3300 1950
-F 0 "#PWR064" H 3300 1800 50  0001 C CNN
+F 0 "#PWR066" H 3300 1800 50  0001 C CNN
 F 1 "+5V" H 3300 2090 50  0000 C CNN
 F 2 "" H 3300 1950 50  0000 C CNN
@@
 $EndComp
 $Comp
-L Earth #PWR065
+L Earth #PWR067
 U 1 1 5BE5344C
 P 3300 2550
-F 0 "#PWR065" H 3300 2300 50  0001 C CNN
+F 0 "#PWR067" H 3300 2300 50  0001 C CNN
 F 1 "Earth" H 3300 2400 50  0001 C CNN
 F 2 "" H 3300 2550 50  0000 C CNN
@@
 Connection ~ 2850 2350
 $Comp
-L Earth #PWR066
+L Earth #PWR068
 U 1 1 5BE53459
 P 3000 1800
-F 0 "#PWR066" H 3000 1550 50  0001 C CNN
+F 0 "#PWR068" H 3000 1550 50  0001 C CNN
 F 1 "Earth" H 3000 1650 50  0001 C CNN
 F 2 "" H 3000 1800 50  0000 C CNN
@@
 F 0 "C601" V 3400 3000 50  0000 L CNN
 F 1 "560pF" V 3300 3000 50  0000 L CNN
-F 2 "Capacitors_THT:C_Axial_L3.8mm_D2.6mm_P7.50mm_Horizontal" H 3388 2800 50  0001 C CNN
+F 2 "Capacitors_SMD:C_0805_HandSoldering" H 3388 2800 50  0001 C CNN
 F 3 "" H 3350 2950 50  0000 C CNN
 	1    3350 2950
@@
 	6900 2350 7250 2350
 $Comp
-L +5V #PWR067
+L +5V #PWR069
 U 1 1 5BE5349B
 P 8250 1950
-F 0 "#PWR067" H 8250 1800 50  0001 C CNN
+F 0 "#PWR069" H 8250 1800 50  0001 C CNN
 F 1 "+5V" H 8250 2090 50  0000 C CNN
 F 2 "" H 8250 1950 50  0000 C CNN
@@
 $EndComp
 $Comp
-L Earth #PWR068
+L Earth #PWR070
 U 1 1 5BE534A1
 P 8250 2550
-F 0 "#PWR068" H 8250 2300 50  0001 C CNN
+F 0 "#PWR070" H 8250 2300 50  0001 C CNN
 F 1 "Earth" H 8250 2400 50  0001 C CNN
 F 2 "" H 8250 2550 50  0000 C CNN
@@
 Connection ~ 7800 2350
 $Comp
-L Earth #PWR069
+L Earth #PWR071
 U 1 1 5BE534AE
 P 7950 1800
-F 0 "#PWR069" H 7950 1550 50  0001 C CNN
+F 0 "#PWR071" H 7950 1550 50  0001 C CNN
 F 1 "Earth" H 7950 1650 50  0001 C CNN
 F 2 "" H 7950 1800 50  0000 C CNN
@@
 F 0 "C602" V 8350 3000 50  0000 L CNN
 F 1 "560pF" V 8250 3000 50  0000 L CNN
-F 2 "Capacitors_THT:C_Axial_L3.8mm_D2.6mm_P7.50mm_Horizontal" H 8338 2800 50  0001 C CNN
+F 2 "Capacitors_SMD:C_0805_HandSoldering" H 8338 2800 50  0001 C CNN
 F 3 "" H 8300 2950 50  0000 C CNN
 	1    8300 2950
@@
 	1950 4600 2300 4600
 $Comp
-L +5V #PWR070
+L +5V #PWR072
 U 1 1 5BE534F7
 P 3300 4200
-F 0 "#PWR070" H 3300 4050 50  0001 C CNN
+F 0 "#PWR072" H 3300 4050 50  0001 C CNN
 F 1 "+5V" H 3300 4340 50  0000 C CNN
 F 2 "" H 3300 4200 50  0000 C CNN
@@
 $EndComp
 $Comp
-L Earth #PWR071
+L Earth #PWR073
 U 1 1 5BE534FD
 P 3300 4800
-F 0 "#PWR071" H 3300 4550 50  0001 C CNN
+F 0 "#PWR073" H 3300 4550 50  0001 C CNN
 F 1 "Earth" H 3300 4650 50  0001 C CNN
 F 2 "" H 3300 4800 50  0000 C CNN
@@
 Connection ~ 2850 4600
 $Comp
-L Earth #PWR072
+L Earth #PWR074
 U 1 1 5BE5350A
 P 3000 4050
-F 0 "#PWR072" H 3000 3800 50  0001 C CNN
+F 0 "#PWR074" H 3000 3800 50  0001 C CNN
 F 1 "Earth" H 3000 3900 50  0001 C CNN
 F 2 "" H 3000 4050 50  0000 C CNN
@@
 F 0 "C603" V 3400 5250 50  0000 L CNN
 F 1 "560pF" V 3300 5250 50  0000 L CNN
-F 2 "Capacitors_THT:C_Axial_L3.8mm_D2.6mm_P7.50mm_Horizontal" H 3388 5050 50  0001 C CNN
+F 2 "Capacitors_SMD:C_0805_HandSoldering" H 3388 5050 50  0001 C CNN
 F 3 "" H 3350 5200 50  0000 C CNN
 	1    3350 5200
@@
 	6900 4600 7250 4600
 $Comp
-L +5V #PWR073
+L +5V #PWR075
 U 1 1 5BE5354C
 P 8250 4200
-F 0 "#PWR073" H 8250 4050 50  0001 C CNN
+F 0 "#PWR075" H 8250 4050 50  0001 C CNN
 F 1 "+5V" H 8250 4340 50  0000 C CNN
 F 2 "" H 8250 4200 50  0000 C CNN
@@
 $EndComp
 $Comp
-L Earth #PWR074
+L Earth #PWR076
 U 1 1 5BE53552
 P 8250 4800
-F 0 "#PWR074" H 8250 4550 50  0001 C CNN
+F 0 "#PWR076" H 8250 4550 50  0001 C CNN
 F 1 "Earth" H 8250 4650 50  0001 C CNN
 F 2 "" H 8250 4800 50  0000 C CNN
@@
 Connection ~ 7800 4600
 $Comp
-L Earth #PWR075
+L Earth #PWR077
 U 1 1 5BE5355F
 P 7950 4050
-F 0 "#PWR075" H 7950 3800 50  0001 C CNN
+F 0 "#PWR077" H 7950 3800 50  0001 C CNN
 F 1 "Earth" H 7950 3900 50  0001 C CNN
 F 2 "" H 7950 4050 50  0000 C CNN
@@
 F 0 "C604" V 8350 5250 50  0000 L CNN
 F 1 "560pF" V 8250 5250 50  0000 L CNN
-F 2 "Capacitors_THT:C_Axial_L3.8mm_D2.6mm_P7.50mm_Horizontal" H 8338 5050 50  0001 C CNN
+F 2 "Capacitors_SMD:C_0805_HandSoldering" H 8338 5050 50  0001 C CNN
 F 3 "" H 8300 5200 50  0000 C CNN
 	1    8300 5200
