File: hardware/buffers 1-4.sch (KiCad schematic (older format))
At the start: 25 parts, among them J301 PJ301M-12, J302 PJ301M-12, J303 PJ301M-12, J304 PJ301M-12, U301 MCP6004

Commit message: jacks on a different sheet than the buffers. single PCB with jumpers and mouse bites
Parts:
- removed J301, J302, J303, J304: PJ301M-12, Eurocad:PJ301M-12, symbol PJ301M-12
- C301, C302, C303, C304: value 330pF -> 560pF; footprint (none) -> Capacitors_THT:C_Axial_L3.8mm_D2.6mm_P7.50mm_Horizontal
- U301: footprint (none) -> Housings_DIP:DIP-14_W7.62mm
- renumbered R305 to R302, R302 to R303, R306 to R304, R303 to R305, R307 to R306, R304 to R307
Connections:
- net in1: now reaches R305.2
- net in2: now reaches R306.2
- net in3: now reaches R313.2
- net in4: now reaches R314.2
- net CV1 renamed out1
- net CV2 renamed out2
- net CV3 renamed out3
- net CV4 renamed out4
Changed lines of the file:
@@
 $Descr A4 11693 8268
 encoding utf-8
-Sheet 3 4
+Sheet 3 6
 Title ""
 Date ""
@@
 Comment4 ""
 $EndDescr
-$Comp
-L PJ301M-12 J301
-U 1 1 5BE21CDD
-P 1550 1800
-F 0 "J301" H 1200 1600 50  0000 C CNN
-F 1 "PJ301M-12" H 1400 2050 50  0000 C CNN
-F 2 "Eurocad:PJ301M-12" H 1550 1800 50  0001 C CNN
-F 3 "" H 1550 1800 50  0000 C CNN
-	1    1550 1800
-	1    0    0    1
-$EndComp
 Text HLabel 2000 1150 0    60   BiDi ~ 0
 -5V
@@
 $EndComp
 $Comp
-L Earth #PWR017
-U 1 1 5BE2619C
-P 2250 2350
-F 0 "#PWR017" H 2250 2100 50  0001 C CNN
-F 1 "Earth" H 2250 2200 50  0001 C CNN
-F 2 "" H 2250 2350 50  0000 C CNN
-F 3 "" H 2250 2350 50  0000 C CNN
-	1    2250 2350
-	1    0    0    -1
-$EndComp
-Wire Wire Line
-	2000 1800 2250 1800
-Wire Wire Line
-	2250 1800 2250 2350
-Wire Wire Line
-	2000 1950 2250 1950
-Connection ~ 2250 1950
-$Comp
-L R R303
+L R R305
 U 1 1 5BE263D1
 P 2500 1700
-F 0 "R303" V 2580 1700 50  0000 C CNN
+F 0 "R305" V 2580 1700 50  0000 C CNN
 F 1 "1k" V 2500 1700 50  0000 C CNN
 F 2 "Resistors_SMD:R_0805_HandSoldering" V 2430 1700 50  0001 C CNN
@@
 	2000 1700 2350 1700
 $Comp
-L +5V #PWR018
+L +5V #PWR021
 U 1 1 5BE268F6
 P 3350 1300
-F 0 "#PWR018" H 3350 1150 50  0001 C CNN
+F 0 "#PWR021" H 3350 1150 50  0001 C CNN
 F 1 "+5V" H 3350 1440 50  0000 C CNN
 F 2 "" H 3350 1300 50  0000 C CNN
@@
 $EndComp
 $Comp
-L Earth #PWR019
+L Earth #PWR022
 U 1 1 5BE26952
 P 3350 1900
-F 0 "#PWR019" H 3350 1650 50  0001 C CNN
+F 0 "#PWR022" H 3350 1650 50  0001 C CNN
 F 1 "Earth" H 3350 1750 50  0001 C CNN
 F 2 "" H 3350 1900 50  0000 C CNN
@@
 Connection ~ 2900 1700
 $Comp
-L Earth #PWR020
+L Earth #PWR023
 U 1 1 5BE271CC
 P 3050 1150
-F 0 "#PWR020" H 3050 900 50  0001 C CNN
+F 0 "#PWR023" H 3050 900 50  0001 C CNN
 F 1 "Earth" H 3050 1000 50  0001 C CNN
 F 2 "" H 3050 1150 50  0000 C CNN
@@
 P 3400 2300
 F 0 "C301" V 3450 2350 50  0000 L CNN
-F 1 "330pF" V 3350 2350 50  0000 L CNN
-F 2 "" H 3438 2150 50  0000 C CNN
+F 1 "560pF" V 3350 2350 50  0000 L CNN
+F 2 "Capacitors_THT:C_Axial_L3.8mm_D2.6mm_P7.50mm_Horizontal" H 3438 2150 50  0001 C CNN
 F 3 "" H 3400 2300 50  0000 C CNN
 	1    3400 2300
@@
 	2900 2300 3250 2300
 $Comp
-L R R304
+L R R307
 U 1 1 5BE276C0
 P 3400 2700
-F 0 "R304" V 3480 2700 50  0000 C CNN
+F 0 "R307" V 3480 2700 50  0000 C CNN
 F 1 "270" V 3400 2700 50  0000 C CNN
 F 2 "Resistors_SMD:R_0805_HandSoldering" V 3330 2700 50  0001 C CNN
@@
 Connection ~ 2900 2300
 $Comp
-L R R302
+L R R303
 U 1 1 5BE278C1
 P 4300 1600
-F 0 "R302" V 4380 1600 50  0000 C CNN
+F 0 "R303" V 4380 1600 50  0000 C CNN
 F 1 "100R" V 4300 1600 50  0000 C CNN
 F 2 "Resistors_SMD:R_0805_HandSoldering" V 4230 1600 50  0001 C CNN
@@
 Connection ~ 3950 2300
 Text HLabel 4850 1150 2    60   Output ~ 0
-CV1
+out1
 Wire Wire Line
 	4450 1600 4700 1600
@@
 Wire Wire Line
 	4700 1150 4850 1150
-$Comp
-L PJ301M-12 J302
-U 1 1 5BE45A40
-P 6500 1800
-F 0 "J302" H 6150 1600 50  0000 C CNN
-F 1 "PJ301M-12" H 6350 2050 50  0000 C CNN
-F 2 "Eurocad:PJ301M-12" H 6500 1800 50  0001 C CNN
-F 3 "" H 6500 1800 50  0000 C CNN
-	1    6500 1800
-	1    0    0    1
-$EndComp
 Text HLabel 6950 1150 0    60   BiDi ~ 0
 -5V
 $Comp
-L Earth #PWR021
-U 1 1 5BE45A4F
-P 7200 2350
-F 0 "#PWR021" H 7200 2100 50  0001 C CNN
-F 1 "Earth" H 7200 2200 50  0001 C CNN
-F 2 "" H 7200 2350 50  0000 C CNN
-F 3 "" H 7200 2350 50  0000 C CNN
-	1    7200 2350
-	1    0    0    -1
-$EndComp
-Wire Wire Line
-	6950 1800 7200 1800
-Wire Wire Line
-	7200 1800 7200 2350
-Wire Wire Line
-	6950 1950 7200 1950
-Connection ~ 7200 1950
-$Comp
-L R R307
+L R R306
 U 1 1 5BE45A5A
 P 7450 1700
-F 0 "R307" V 7530 1700 50  0000 C CNN
+F 0 "R306" V 7530 1700 50  0000 C CNN
 F 1 "1k" V 7450 1700 50  0000 C CNN
 F 2 "Resistors_SMD:R_0805_HandSoldering" V 7380 1700 50  0001 C CNN
@@
 $EndComp
 $Comp
-L R R305
+L R R302
 U 1 1 5BE45A62
 P 7450 1350
-F 0 "R305" V 7530 1350 50  0000 C CNN
+F 0 "R302" V 7530 1350 50  0000 C CNN
 F 1 "499" V 7450 1350 50  0000 C CNN
 F 2 "Resistors_SMD:R_0805_HandSoldering" V 7380 1350 50  0001 C CNN
@@
 	6950 1700 7300 1700
 $Comp
-L +5V #PWR022
+L +5V #PWR024
 U 1 1 5BE45A6C
 P 8300 1300
-F 0 "#PWR022" H 8300 1150 50  0001 C CNN
+F 0 "#PWR024" H 8300 1150 50  0001 C CNN
 F 1 "+5V" H 8300 1440 50  0000 C CNN
 F 2 "" H 8300 1300 50  0000 C CNN
@@
 $EndComp
 $Comp
-L Earth #PWR023
+L Earth #PWR025
 U 1 1 5BE45A72
 P 8300 1900
-F 0 "#PWR023" H 8300 1650 50  0001 C CNN
+F 0 "#PWR025" H 8300 1650 50  0001 C CNN
 F 1 "Earth" H 8300 1750 50  0001 C CNN
 F 2 "" H 8300 1900 50  0000 C CNN
@@
 Connection ~ 7850 1700
 $Comp
-L Earth #PWR024
+L Earth #PWR026
 U 1 1 5BE45A7C
 P 8000 1150
-F 0 "#PWR024" H 8000 900 50  0001 C CNN
+F 0 "#PWR026" H 8000 900 50  0001 C CNN
 F 1 "Earth" H 8000 1000 50  0001 C CNN
 F 2 "" H 8000 1150 50  0000 C CNN
@@
 P 8350 2300
 F 0 "C302" V 8400 2350 50  0000 L CNN
-F 1 "330pF" V 8300 2350 50  0000 L CNN
-F 2 "" H 8388 2150 50  0000 C CNN
+F 1 "560pF" V 8300 2350 50  0000 L CNN
+F 2 "Capacitors_THT:C_Axial_L3.8mm_D2.6mm_P7.50mm_Horizontal" H 8388 2150 50  0001 C CNN
 F 3 "" H 8350 2300 50  0000 C CNN
 	1    8350 2300
@@
 Connection ~ 7850 2300
 $Comp
-L R R306
+L R R304
 U 1 1 5BE45A97
 P 9250 1600
-F 0 "R306" V 9330 1600 50  0000 C CNN
+F 0 "R304" V 9330 1600 50  0000 C CNN
 F 1 "100R" V 9250 1600 50  0000 C CNN
 F 2 "Resistors_SMD:R_0805_HandSoldering" V 9180 1600 50  0001 C CNN
@@
 Connection ~ 8900 2300
 Text HLabel 9800 1150 2    60   Output ~ 0
-CV2
+out2
 Wire Wire Line
 	9400 1600 9650 1600
@@
 F 0 "U301" H 8400 1800 50  0000 L CNN
 F 1 "MCP6004" H 8400 1400 50  0000 L CNN
-F 2 "" H 8350 1700 50  0000 C CNN
+F 2 "Housings_DIP:DIP-14_W7.62mm" H 8350 1700 50  0001 C CNN
 F 3 "" H 8450 1800 50  0000 C CNN
 	2    8400 1600
 	1    0    0    -1
 $EndComp
-$Comp
-L PJ301M-12 J303
-U 1 1 5BE4605B
-P 1550 4050
-F 0 "J303" H 1200 3850 50  0000 C CNN
-F 1 "PJ301M-12" H 1400 4300 50  0000 C CNN
-F 2 "Eurocad:PJ301M-12" H 1550 4050 50  0001 C CNN
-F 3 "" H 1550 4050 50  0000 C CNN
-	1    1550 4050
-	1    0    0    1
-$EndComp
 Text HLabel 2000 3400 0    60   BiDi ~ 0
 -5V
-$Comp
-L Earth #PWR025
-U 1 1 5BE4606A
-P 2250 4600
-F 0 "#PWR025" H 2250 4350 50  0001 C CNN
-F 1 "Earth" H 2250 4450 50  0001 C CNN
-F 2 "" H 2250 4600 50  0000 C CNN
-F 3 "" H 2250 4600 50  0000 C CNN
-	1    2250 4600
-	1    0    0    -1
-$EndComp
-Wire Wire Line
-	2000 4050 2250 4050
-Wire Wire Line
-	2250 4050 2250 4600
-Wire Wire Line
-	2000 4200 2250 4200
-Connection ~ 2250 4200
 $Comp
 L R R313
@@
 	2000 3950 2350 3950
 $Comp
-L +5V #PWR026
+L +5V #PWR027
 U 1 1 5BE46087
 P 3350 3550
-F 0 "#PWR026" H 3350 3400 50  0001 C CNN
+F 0 "#PWR027" H 3350 3400 50  0001 C CNN
 F 1 "+5V" H 3350 3690 50  0000 C CNN
 F 2 "" H 3350 3550 50  0000 C CNN
@@
 $EndComp
 $Comp
-L Earth #PWR027
+L Earth #PWR028
 U 1 1 5BE4608D
 P 3350 4150
-F 0 "#PWR027" H 3350 3900 50  0001 C CNN
+F 0 "#PWR028" H 3350 3900 50  0001 C CNN
 F 1 "Earth" H 3350 4000 50  0001 C CNN
 F 2 "" H 3350 4150 50  0000 C CNN
@@
 Connection ~ 2900 3950
 $Comp
-L Earth #PWR028
+L Earth #PWR029
 U 1 1 5BE46097
 P 3050 3400
-F 0 "#PWR028" H 3050 3150 50  0001 C CNN
+F 0 "#PWR029" H 3050 3150 50  0001 C CNN
 F 1 "Earth" H 3050 3250 50  0001 C CNN
 F 2 "" H 3050 3400 50  0000 C CNN
@@
 P 3400 4550
 F 0 "C303" V 3450 4600 50  0000 L CNN
-F 1 "330pF" V 3350 4600 50  0000 L CNN
-F 2 "" H 3438 4400 50  0000 C CNN
+F 1 "560pF" V 3350 4600 50  0000 L CNN
+F 2 "Capacitors_THT:C_Axial_L3.8mm_D2.6mm_P7.50mm_Horizontal" H 3438 4400 50  0001 C CNN
 F 3 "" H 3400 4550 50  0000 C CNN
 	1    3400 4550
@@
 Connection ~ 3950 4550
 Text HLabel 4850 3400 2    60   Output ~ 0
-CV3
+out3
 Wire Wire Line
 	4450 3850 4700 3850
@@
 Wire Wire Line
 	4700 3400 4850 3400
-$Comp
-L PJ301M-12 J304
-U 1 1 5BE46489
-P 6500 4050
-F 0 "J304" H 6150 3850 50  0000 C CNN
-F 1 "PJ301M-12" H 6350 4300 50  0000 C CNN
-F 2 "Eurocad:PJ301M-12" H 6500 4050 50  0001 C CNN
-F 3 "" H 6500 4050 50  0000 C CNN
-	1    6500 4050
-	1    0    0    1
-$EndComp
 Text HLabel 6950 3400 0    60   BiDi ~ 0
 -5V
-$Comp
-L Earth #PWR029
-U 1 1 5BE46498
-P 7200 4600
-F 0 "#PWR029" H 7200 4350 50  0001 C CNN
-F 1 "Earth" H 7200 4450 50  0001 C CNN
-F 2 "" H 7200 4600 50  0000 C CNN
-F 3 "" H 7200 4600 50  0000 C CNN
-	1    7200 4600
-	1    0    0    -1
-$EndComp
-Wire Wire Line
-	6950 4050 7200 4050
-Wire Wire Line
-	7200 4050 7200 4600
-Wire Wire Line
-	6950 4200 7200 4200
-Connection ~ 7200 4200
 $Comp
 L R R314
@@
 P 8350 4550
 F 0 "C304" V 8400 4600 50  0000 L CNN
-F 1 "330pF" V 8300 4600 50  0000 L CNN
-F 2 "" H 8388 4400 50  0000 C CNN
+F 1 "560pF" V 8300 4600 50  0000 L CNN
+F 2 "Capacitors_THT:C_Axial_L3.8mm_D2.6mm_P7.50mm_Horizontal" H 8388 4400 50  0001 C CNN
 F 3 "" H 8350 4550 50  0000 C CNN
 	1    8350 4550
@@
 Connection ~ 8900 4550
 Text HLabel 9800 3400 2    60   Output ~ 0
-CV4
+out4
 Wire Wire Line
 	9400 3850 9650 3850
@@
 F 0 "U301" H 8400 4050 50  0000 L CNN
 F 1 "MCP6004" H 8400 3650 50  0000 L CNN
-F 2 "" H 8350 3950 50  0000 C CNN
+F 2 "Housings_DIP:DIP-14_W7.62mm" H 8350 3950 50  0001 C CNN
 F 3 "" H 8450 4050 50  0000 C CNN
 	4    8400 3850
@@
 F 0 "U301" H 3450 4050 50  0000 L CNN
 F 1 "MCP6004" H 3450 3650 50  0000 L CNN
-F 2 "" H 3400 3950 50  0000 C CNN
+F 2 "Housings_DIP:DIP-14_W7.62mm" H 3400 3950 50  0001 C CNN
 F 3 "" H 3500 4050 50  0000 C CNN
 	3    3450 3850
 	1    0    0    -1
 $EndComp
+Text HLabel 2000 3950 0    60   Input ~ 0
+in3
+Text HLabel 2000 1700 0    60   Input ~ 0
+in1
+Text HLabel 6950 1700 0    60   Input ~ 0
+in2
+Text HLabel 6950 3950 0    60   Input ~ 0
+in4
 $EndSCHEMATC

Commit message: most of the scematic is complete with the exception of the -5V offset
Parts:
- U301: footprint Housings_DIP:DIP-14_W7.62mm -> Housings_SOIC:SOIC-14_3.9x8.7mm_Pitch1.27mm
Changed lines of the file:
@@
 F 0 "U301" H 3450 1800 50  0000 L CNN
 F 1 "MCP6004" H 3450 1400 50  0000 L CNN
-F 2 "Housings_DIP:DIP-14_W7.62mm" H 3400 1700 50  0001 C CNN
+F 2 "Housings_SOIC:SOIC-14_3.9x8.7mm_Pitch1.27mm" H 3400 1700 50  0001 C CNN
 F 3 "" H 3500 1800 50  0000 C CNN
 	1    3450 1600
@@
 	2000 1700 2350 1700
 $Comp
-L +5V #PWR021
+L +5V #PWR025
 U 1 1 5BE268F6
 P 3350 1300
-F 0 "#PWR021" H 3350 1150 50  0001 C CNN
+F 0 "#PWR025" H 3350 1150 50  0001 C CNN
 F 1 "+5V" H 3350 1440 50  0000 C CNN
 F 2 "" H 3350 1300 50  0000 C CNN
@@
 $EndComp
 $Comp
-L Earth #PWR022
+L Earth #PWR026
 U 1 1 5BE26952
 P 3350 1900
-F 0 "#PWR022" H 3350 1650 50  0001 C CNN
+F 0 "#PWR026" H 3350 1650 50  0001 C CNN
 F 1 "Earth" H 3350 1750 50  0001 C CNN
 F 2 "" H 3350 1900 50  0000 C CNN
@@
 Connection ~ 2900 1700
 $Comp
-L Earth #PWR023
+L Earth #PWR027
 U 1 1 5BE271CC
 P 3050 1150
-F 0 "#PWR023" H 3050 900 50  0001 C CNN
+F 0 "#PWR027" H 3050 900 50  0001 C CNN
 F 1 "Earth" H 3050 1000 50  0001 C CNN
 F 2 "" H 3050 1150 50  0000 C CNN
@@
 	6950 1700 7300 1700
 $Comp
-L +5V #PWR024
+L +5V #PWR028
 U 1 1 5BE45A6C
 P 8300 1300
-F 0 "#PWR024" H 8300 1150 50  0001 C CNN
+F 0 "#PWR028" H 8300 1150 50  0001 C CNN
 F 1 "+5V" H 8300 1440 50  0000 C CNN
 F 2 "" H 8300 1300 50  0000 C CNN
@@
 $EndComp
 $Comp
-L Earth #PWR025
+L Earth #PWR029
 U 1 1 5BE45A72
 P 8300 1900
-F 0 "#PWR025" H 8300 1650 50  0001 C CNN
+F 0 "#PWR029" H 8300 1650 50  0001 C CNN
 F 1 "Earth" H 8300 1750 50  0001 C CNN
 F 2 "" H 8300 1900 50  0000 C CNN
@@
 Connection ~ 7850 1700
 $Comp
-L Earth #PWR026
+L Earth #PWR030
 U 1 1 5BE45A7C
 P 8000 1150
-F 0 "#PWR026" H 8000 900 50  0001 C CNN
+F 0 "#PWR030" H 8000 900 50  0001 C CNN
 F 1 "Earth" H 8000 1000 50  0001 C CNN
 F 2 "" H 8000 1150 50  0000 C CNN
@@
 F 0 "U301" H 8400 1800 50  0000 L CNN
 F 1 "MCP6004" H 8400 1400 50  0000 L CNN
-F 2 "Housings_DIP:DIP-14_W7.62mm" H 8350 1700 50  0001 C CNN
+F 2 "Housings_SOIC:SOIC-14_3.9x8.7mm_Pitch1.27mm" H 8350 1700 50  0001 C CNN
 F 3 "" H 8450 1800 50  0000 C CNN
 	2    8400 1600
@@
 	2000 3950 2350 3950
 $Comp
-L +5V #PWR027
+L +5V #PWR031
 U 1 1 5BE46087
 P 3350 3550
-F 0 "#PWR027" H 3350 3400 50  0001 C CNN
+F 0 "#PWR031" H 3350 3400 50  0001 C CNN
 F 1 "+5V" H 3350 3690 50  0000 C CNN
 F 2 "" H 3350 3550 50  0000 C CNN
@@
 $EndComp
 $Comp
-L Earth #PWR028
+L Earth #PWR032
 U 1 1 5BE4608D
 P 3350 4150
-F 0 "#PWR028" H 3350 3900 50  0001 C CNN
+F 0 "#PWR032" H 3350 3900 50  0001 C CNN
 F 1 "Earth" H 3350 4000 50  0001 C CNN
 F 2 "" H 3350 4150 50  0000 C CNN
@@
 Connection ~ 2900 3950
 $Comp
-L Earth #PWR029
+L Earth #PWR033
 U 1 1 5BE46097
 P 3050 3400
-F 0 "#PWR029" H 3050 3150 50  0001 C CNN
+F 0 "#PWR033" H 3050 3150 50  0001 C CNN
 F 1 "Earth" H 3050 3250 50  0001 C CNN
 F 2 "" H 3050 3400 50  0000 C CNN
@@
 	6950 3950 7300 3950
 $Comp
-L +5V #PWR030
+L +5V #PWR034
 U 1 1 5BE464B5
 P 8300 3550
-F 0 "#PWR030" H 8300 3400 50  0001 C CNN
+F 0 "#PWR034" H 8300 3400 50  0001 C CNN
 F 1 "+5V" H 8300 3690 50  0000 C CNN
 F 2 "" H 8300 3550 50  0000 C CNN
@@
 $EndComp
 $Comp
-L Earth #PWR031
+L Earth #PWR035
 U 1 1 5BE464BB
 P 8300 4150
-F 0 "#PWR031" H 8300 3900 50  0001 C CNN
+F 0 "#PWR035" H 8300 3900 50  0001 C CNN
 F 1 "Earth" H 8300 4000 50  0001 C CNN
 F 2 "" H 8300 4150 50  0000 C CNN
@@
 Connection ~ 7850 3950
 $Comp
-L Earth #PWR032
+L Earth #PWR036
 U 1 1 5BE464C5
 P 8000 3400
-F 0 "#PWR032" H 8000 3150 50  0001 C CNN
+F 0 "#PWR036" H 8000 3150 50  0001 C CNN
 F 1 "Earth" H 8000 3250 50  0001 C CNN
 F 2 "" H 8000 3400 50  0000 C CNN
@@
 F 0 "U301" H 8400 4050 50  0000 L CNN
 F 1 "MCP6004" H 8400 3650 50  0000 L CNN
-F 2 "Housings_DIP:DIP-14_W7.62mm" H 8350 3950 50  0001 C CNN
+F 2 "Housings_SOIC:SOIC-14_3.9x8.7mm_Pitch1.27mm" H 8350 3950 50  0001 C CNN
 F 3 "" H 8450 4050 50  0000 C CNN
 	4    8400 3850
@@
 F 0 "U301" H 3450 4050 50  0000 L CNN
 F 1 "MCP6004" H 3450 3650 50  0000 L CNN
-F 2 "Housings_DIP:DIP-14_W7.62mm" H 3400 3950 50  0001 C CNN
+F 2 "Housings_SOIC:SOIC-14_3.9x8.7mm_Pitch1.27mm" H 3400 3950 50  0001 C CNN
 F 3 "" H 3500 4050 50  0000 C CNN
 	3    3450 3850

Commit message: updated footprint & first tracks laid
Parts:
- C301, C302, C303, C304: footprint Capacitors_THT:C_Axial_L3.8mm_D2.6mm_P7.50mm_Horizontal -> Capacitors_SMD:C_0805_HandSoldering
Changed lines of the file:
@@
 	2000 1700 2350 1700
 $Comp
-L +5V #PWR025
+L +5V #PWR027
 U 1 1 5BE268F6
 P 3350 1300
-F 0 "#PWR025" H 3350 1150 50  0001 C CNN
+F 0 "#PWR027" H 3350 1150 50  0001 C CNN
 F 1 "+5V" H 3350 1440 50  0000 C CNN
 F 2 "" H 3350 1300 50  0000 C CNN
@@
 $EndComp
 $Comp
-L Earth #PWR026
+L Earth #PWR028
 U 1 1 5BE26952
 P 3350 1900
-F 0 "#PWR026" H 3350 1650 50  0001 C CNN
+F 0 "#PWR028" H 3350 1650 50  0001 C CNN
 F 1 "Earth" H 3350 1750 50  0001 C CNN
 F 2 "" H 3350 1900 50  0000 C CNN
@@
 Connection ~ 2900 1700
 $Comp
-L Earth #PWR027
+L Earth #PWR029
 U 1 1 5BE271CC
 P 3050 1150
-F 0 "#PWR027" H 3050 900 50  0001 C CNN
+F 0 "#PWR029" H 3050 900 50  0001 C CNN
 F 1 "Earth" H 3050 1000 50  0001 C CNN
 F 2 "" H 3050 1150 50  0000 C CNN
@@
 F 0 "C301" V 3450 2350 50  0000 L CNN
 F 1 "560pF" V 3350 2350 50  0000 L CNN
-F 2 "Capacitors_THT:C_Axial_L3.8mm_D2.6mm_P7.50mm_Horizontal" H 3438 2150 50  0001 C CNN
+F 2 "Capacitors_SMD:C_0805_HandSoldering" H 3438 2150 50  0001 C CNN
 F 3 "" H 3400 2300 50  0000 C CNN
 	1    3400 2300
@@
 	6950 1700 7300 1700
 $Comp
-L +5V #PWR028
+L +5V #PWR030
 U 1 1 5BE45A6C
 P 8300 1300
-F 0 "#PWR028" H 8300 1150 50  0001 C CNN
+F 0 "#PWR030" H 8300 1150 50  0001 C CNN
 F 1 "+5V" H 8300 1440 50  0000 C CNN
 F 2 "" H 8300 1300 50  0000 C CNN
@@
 $EndComp
 $Comp
-L Earth #PWR029
+L Earth #PWR031
 U 1 1 5BE45A72
 P 8300 1900
-F 0 "#PWR029" H 8300 1650 50  0001 C CNN
+F 0 "#PWR031" H 8300 1650 50  0001 C CNN
 F 1 "Earth" H 8300 1750 50  0001 C CNN
 F 2 "" H 8300 1900 50  0000 C CNN
@@
 Connection ~ 7850 1700
 $Comp
-L Earth #PWR030
+L Earth #PWR032
 U 1 1 5BE45A7C
 P 8000 1150
-F 0 "#PWR030" H 8000 900 50  0001 C CNN
+F 0 "#PWR032" H 8000 900 50  0001 C CNN
 F 1 "Earth" H 8000 1000 50  0001 C CNN
 F 2 "" H 8000 1150 50  0000 C CNN
@@
 F 0 "C302" V 8400 2350 50  0000 L CNN
 F 1 "560pF" V 8300 2350 50  0000 L CNN
-F 2 "Capacitors_THT:C_Axial_L3.8mm_D2.6mm_P7.50mm_Horizontal" H 8388 2150 50  0001 C CNN
+F 2 "Capacitors_SMD:C_0805_HandSoldering" H 8388 2150 50  0001 C CNN
 F 3 "" H 8350 2300 50  0000 C CNN
 	1    8350 2300
@@
 	2000 3950 2350 3950
 $Comp
-L +5V #PWR031
+L +5V #PWR033
 U 1 1 5BE46087
 P 3350 3550
-F 0 "#PWR031" H 3350 3400 50  0001 C CNN
+F 0 "#PWR033" H 3350 3400 50  0001 C CNN
 F 1 "+5V" H 3350 3690 50  0000 C CNN
 F 2 "" H 3350 3550 50  0000 C CNN
@@
 $EndComp
 $Comp
-L Earth #PWR032
+L Earth #PWR034
 U 1 1 5BE4608D
 P 3350 4150
-F 0 "#PWR032" H 3350 3900 50  0001 C CNN
+F 0 "#PWR034" H 3350 3900 50  0001 C CNN
 F 1 "Earth" H 3350 4000 50  0001 C CNN
 F 2 "" H 3350 4150 50  0000 C CNN
@@
 Connection ~ 2900 3950
 $Comp
-L Earth #PWR033
+L Earth #PWR035
 U 1 1 5BE46097
 P 3050 3400
-F 0 "#PWR033" H 3050 3150 50  0001 C CNN
+F 0 "#PWR035" H 3050 3150 50  0001 C CNN
 F 1 "Earth" H 3050 3250 50  0001 C CNN
 F 2 "" H 3050 3400 50  0000 C CNN
@@
 F 0 "C303" V 3450 4600 50  0000 L CNN
 F 1 "560pF" V 3350 4600 50  0000 L CNN
-F 2 "Capacitors_THT:C_Axial_L3.8mm_D2.6mm_P7.50mm_Horizontal" H 3438 4400 50  0001 C CNN
+F 2 "Capacitors_SMD:C_0805_HandSoldering" H 3438 4400 50  0001 C CNN
 F 3 "" H 3400 4550 50  0000 C CNN
 	1    3400 4550
@@
 	6950 3950 7300 3950
 $Comp
-L +5V #PWR034
+L +5V #PWR036
 U 1 1 5BE464B5
 P 8300 3550
-F 0 "#PWR034" H 8300 3400 50  0001 C CNN
+F 0 "#PWR036" H 8300 3400 50  0001 C CNN
 F 1 "+5V" H 8300 3690 50  0000 C CNN
 F 2 "" H 8300 3550 50  0000 C CNN
@@
 $EndComp
 $Comp
-L Earth #PWR035
+L Earth #PWR037
 U 1 1 5BE464BB
 P 8300 4150
-F 0 "#PWR035" H 8300 3900 50  0001 C CNN
+F 0 "#PWR037" H 8300 3900 50  0001 C CNN
 F 1 "Earth" H 8300 4000 50  0001 C CNN
 F 2 "" H 8300 4150 50  0000 C CNN
@@
 Connection ~ 7850 3950
 $Comp
-L Earth #PWR036
+L Earth #PWR038
 U 1 1 5BE464C5
 P 8000 3400
-F 0 "#PWR036" H 8000 3150 50  0001 C CNN
+F 0 "#PWR038" H 8000 3150 50  0001 C CNN
 F 1 "Earth" H 8000 3250 50  0001 C CNN
 F 2 "" H 8000 3400 50  0000 C CNN
@@
 F 0 "C304" V 8400 4600 50  0000 L CNN
 F 1 "560pF" V 8300 4600 50  0000 L CNN
-F 2 "Capacitors_THT:C_Axial_L3.8mm_D2.6mm_P7.50mm_Horizontal" H 8388 4400 50  0001 C CNN
+F 2 "Capacitors_SMD:C_0805_HandSoldering" H 8388 4400 50  0001 C CNN
 F 3 "" H 8350 4550 50  0000 C CNN
 	1    8350 4550

Commit message: rotated first op amp & shofted 40-pin connector to match 3d model
Connections:
- net at C301.1, R303.2, R307.1: now also U301.14; no longer U301.1
- net at C301.2, R301.1, R305.1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: now also U301.13 (-); no longer U301.2 (-)
- net at C302.2, R302.1, R306.1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: now also U301.9 (-); no longer U301.6 (-)
- net at C302.1, R304.2, R308.1: now also U301.8; no longer U301.7
- net at C303.2, R309.1, R313.1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: now also U301.6 (-); no longer U301.9 (-)
- net at C303.1, R311.2, R315.1: now also U301.7; no longer U301.8
- net at C304.2, R310.1, R314.1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: now also U301.2 (-); no longer U301.13 (-)
- net at C304.1, R312.2, R316.1: now also U301.1; no longer U301.14
Other:
- moved on the sheet: U301A, U301B, U301C, U301D
Changed lines of the file:
@@
 L MCP6004 U301
 U 1 1 5BE25FAF
-P 3450 1600
-F 0 "U301" H 3450 1800 50  0000 L CNN
-F 1 "MCP6004" H 3450 1400 50  0000 L CNN
-F 2 "Housings_SOIC:SOIC-14_3.9x8.7mm_Pitch1.27mm" H 3400 1700 50  0001 C CNN
-F 3 "" H 3500 1800 50  0000 C CNN
-	1    3450 1600
+P 8400 3850
+F 0 "U301" H 8400 4050 50  0000 L CNN
+F 1 "MCP6004" H 8400 3650 50  0000 L CNN
+F 2 "Housings_SOIC:SOIC-14_3.9x8.7mm_Pitch1.27mm" H 8350 3950 50  0001 C CNN
+F 3 "" H 8450 4050 50  0000 C CNN
+	1    8400 3850
 	1    0    0    -1
 $EndComp
@@
 L MCP6004 U301
 U 2 1 5BE45CBD
-P 8400 1600
-F 0 "U301" H 8400 1800 50  0000 L CNN
-F 1 "MCP6004" H 8400 1400 50  0000 L CNN
-F 2 "Housings_SOIC:SOIC-14_3.9x8.7mm_Pitch1.27mm" H 8350 1700 50  0001 C CNN
-F 3 "" H 8450 1800 50  0000 C CNN
-	2    8400 1600
+P 3450 3850
+F 0 "U301" H 3450 4050 50  0000 L CNN
+F 1 "MCP6004" H 3450 3650 50  0000 L CNN
+F 2 "Housings_SOIC:SOIC-14_3.9x8.7mm_Pitch1.27mm" H 3400 3950 50  0001 C CNN
+F 3 "" H 3500 4050 50  0000 C CNN
+	2    3450 3850
 	1    0    0    -1
 $EndComp
@@
 L MCP6004 U301
 U 4 1 5BE46804
-P 8400 3850
-F 0 "U301" H 8400 4050 50  0000 L CNN
-F 1 "MCP6004" H 8400 3650 50  0000 L CNN
-F 2 "Housings_SOIC:SOIC-14_3.9x8.7mm_Pitch1.27mm" H 8350 3950 50  0001 C CNN
-F 3 "" H 8450 4050 50  0000 C CNN
-	4    8400 3850
+P 3450 1600
+F 0 "U301" H 3450 1800 50  0000 L CNN
+F 1 "MCP6004" H 3450 1400 50  0000 L CNN
+F 2 "Housings_SOIC:SOIC-14_3.9x8.7mm_Pitch1.27mm" H 3400 1700 50  0001 C CNN
+F 3 "" H 3500 1800 50  0000 C CNN
+	4    3450 1600
 	1    0    0    -1
 $EndComp
@@
 L MCP6004 U301
 U 3 1 5BE46A33
-P 3450 3850
-F 0 "U301" H 3450 4050 50  0000 L CNN
-F 1 "MCP6004" H 3450 3650 50  0000 L CNN
-F 2 "Housings_SOIC:SOIC-14_3.9x8.7mm_Pitch1.27mm" H 3400 3950 50  0001 C CNN
-F 3 "" H 3500 4050 50  0000 C CNN
-	3    3450 3850
-	1    0    0    -1
-$EndComp
+P 8400 1600
+F 0 "U301" H 8400 1800 50  0000 L CNN
+F 1 "MCP6004" H 8400 1400 50  0000 L CNN
+F 2 "Housings_SOIC:SOIC-14_3.9x8.7mm_Pitch1.27mm" H 8350 1700 50  0001 C CNN
+F 3 "" H 8450 1800 50  0000 C CNN
+	3    8400 1600
+	1    0    0    -1
+$EndComp
